Commit message: files updated

File: description/robot_core.xacro (robot description, xacro)
@@ -1,4 +1,5 @@
 <?xml version="1.0"?>
 <robot xmlns:xacro="http://www.ros.org/wiki/xacro">
+    <xacro:include filename="inertial_macros.xacro"/>
     <material name="white">
         <color rgba="1 1 1 1"/>
@@ -19,45 +20,116 @@
     <joint name="chassis_joint" type="fixed">
         <parent link="base_link"/>
-        <child link ="chassis"/>
+        <child link="chassis"/>
         <origin xyz="-0.12 0 0"/>
     </joint>
-     <link name="chassis">
+    <link name="chassis">
         <visual>
             <origin xyz="0.11275 0 0.024"/>
             <geometry>
-                <box size="0.2255 .16 .048"/>
+                <box size="0.2255 0.16 .048"/>
             </geometry>
             <material name="white"/>
         </visual>
-     </link>
-     <!-- LEFT WHEEL LINK -->
-     <joint name="left_wheel_joint" type="continuous">
+        <collision>
+            <origin xyz="0.11275 0 0.024"/>
+            <geometry>
+                <box size="0.2255 0.16 .048"/>
+            </geometry>
+        </collision>
+        <xacro:inertial_box mass="0.58" x="0.2255" y="0.16" z="0.048">
+            <origin xyz="0.11275 0 0.024" rpy="0 0 0"/>
+        </xacro:inertial_box>
+    </link>
+    <!-- LEFT BACKWARD WHEEL LINK -->
+    <joint name="left_backward_wheel_joint" type="continuous">
         <parent link="base_link"/>
-        <child link ="left_wheel"/>
+        <child link="left_backward_wheel"/>
         <origin xyz="-0.08475 0.093 0" rpy="-${pi/2} 0 0"/>
-         <axis xyz="0 0 1"/>
-     </joint>
-     <link name="left_wheel">
+        <axis xyz="0 0 1"/>
+    </joint>
+    <link name="left_backward_wheel">
         <visual>
             <geometry>
-                 <cylinder radius="0.0415" length="0.035"/>
+                <cylinder radius="0.0415" length="0.035"/>
             </geometry>
             <material name="blue"/>
         </visual>
-     </link>
-     <!-- RIGHT WHEEL LINK -->
-     <joint name="right_wheel_joint" type="continuous">
+        <collision>
+            <geometry>
+                <cylinder radius="0.0415" length="0.035"/>
+            </geometry>
+        </collision>
+        <xacro:inertial_cylinder mass="0.057" length="0.035" radius="0.0415">
+            <origin xyz="0 0 0" rpy="0 0 0"/>
+        </xacro:inertial_cylinder>
+    </link>
+    <!-- RIGHT BACKWARD WHEEL LINK -->
+    <joint name="right_backward_wheel_joint" type="continuous">
         <parent link="base_link"/>
-        <child link ="right_wheel"/>
+        <child link="right_backward_wheel"/>
         <origin xyz="-0.08475 -0.093 0" rpy="${pi/2} 0 0"/>
-         <axis xyz="0 0 -"/>
-     </joint>
-     <link name="right_wheel">
+        <axis xyz="0 0 -1"/>
+    </joint>
+    <link name="right_backward_wheel">
         <visual>
             <geometry>
-                 <cylinder radius="0.0415" length="0.035"/>
+                <cylinder radius="0.0415" length="0.035"/>
             </geometry>
             <material name="blue"/>
         </visual>
-     </link>
+        <collision>
+            <geometry>
+                <cylinder radius="0.0415" length="0.035"/>
+            </geometry>
+        </collision>
+        <xacro:inertial_cylinder mass="0.057" length="0.035" radius="0.0415">
+            <origin xyz="0 0 0" rpy="0 0 0"/>
+        </xacro:inertial_cylinder>
+    </link>
+    <!-- LEFT FORWARD WHEEL LINK -->
+    <joint name="left_forward_wheel_joint" type="continuous">
+        <parent link="base_link"/>
+        <child link="left_forward_wheel"/>
+        <origin xyz="0.08475 0.093 0" rpy="-${pi/2} 0 0"/>
+        <axis xyz="0 0 1"/>
+    </joint>
+    <link name="left_forward_wheel">
+        <visual>
+            <geometry>
+                <cylinder radius="0.0415" length="0.035"/>
+            </geometry>
+            <material name="blue"/>
+        </visual>
+        <collision>
+            <geometry>
+                <cylinder radius="0.0415" length="0.035"/>
+            </geometry>
+        </collision>
+        <xacro:inertial_cylinder mass="0.057" length="0.035" radius="0.0415">
+            <origin xyz="0 0 0" rpy="0 0 0"/>
+        </xacro:inertial_cylinder>
+    </link>
+    <!-- RIGHT FORWARD WHEEL LINK -->
+    <joint name="right_forward_wheel_joint" type="continuous">
+        <parent link="base_link"/>
+        <child link="right_forward_wheel"/>
+        <origin xyz="0.08475 -0.093 0" rpy="${pi/2} 0 0"/>
+        <axis xyz="0 0 -1"/>
+    </joint>
+    <link name="right_forward_wheel">
+        <visual>
+            <geometry>
+                <cylinder radius="0.0415" length="0.035"/>
+            </geometry>
+            <material name="blue"/>
+        </visual>
+        <collision >
+            <geometry>
+                <cylinder radius="0.0415" length="0.035"/>
+            </geometry>
+        </collision>
+        <xacro:inertial_cylinder mass="0.057" length="0.035" radius="0.0415">
+            <origin xyz="0 0 0" rpy="0 0 0"/>
+        </xacro:inertial_cylinder>
+    </link>
 </robot>
